File: the PETER switchplate.kicad_pcb (KiCad board)
At the start: 2 copper layers, 241.6 x 96.9 mm, 9 parts, among them SW1 RotaryEncoder_Switch, SW12 RotaryEncoder_Switch

Commit message: switchplate clean up
Parts:
- moved G*** 10.2 mm to (141.5, 67.9)
Changed lines of the file:
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@@
   )
   (footprint "LOGO" (layer "F.Cu")
-    (at 140.716 57.785)
+    (at 141.478 67.945)
     (attr board_only exclude_from_pos_files exclude_from_bom)
     (fp_text reference "G***" (at 0 0) (layer "F.SilkS")

Commit message: generate gerber for plate file
Parts:
- removed MX1, MX12: MX-NoLED, MX_Only:MXOnly-1U-NoLED
- removed SW1, SW12: RotaryEncoder_Switch, Keebio-Parts:RotaryEncoder_Alps_EC11E-Switch_Vertical_H20mm

Commit message: planning m2 holes and relief cuts
Parts:
- moved REF** 21.6 mm to (68.2, 49.7)
- moved REF** 21.5 mm to (220.6, 49.5)
- moved REF** 3.56 mm to (244.5, 141.0)
- moved REF** 2.80 mm to (47.8, 140.2)
Other:
- board text added: "make sure m2 are where they need to be!"
Changed lines of the file:
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@@
   (net 0 "")
   (footprint "MountingHole:MountingHole_2.2mm_M2_Pad" (layer "F.Cu")
-    (at 47.879 137.414)
+    (at 47.752 140.208)
     (descr "Mounting Hole 2.2mm, M2")
     (tags "mounting hole 2.2mm m2")
@@
   )
   (footprint "MountingHole:MountingHole_2.2mm_M2_Pad" (layer "F.Cu")
-    (at 244.475 137.414)
+    (at 244.475 140.97)
     (descr "Mounting Hole 2.2mm, M2")
     (tags "mounting hole 2.2mm m2")
@@
   )
   (footprint "MountingHole:MountingHole_2.2mm_M2_Pad" (layer "F.Cu")
-    (at 241.935 51.943)
+    (at 220.599 49.53)
     (descr "Mounting Hole 2.2mm, M2")
     (tags "mounting hole 2.2mm m2")
@@
   )
   (footprint "MountingHole:MountingHole_2.2mm_M2_Pad" (layer "F.Cu")
-    (at 46.736 52.07)
+    (at 68.199 49.657)
     (descr "Mounting Hole 2.2mm, M2")
     (tags "mounting hole 2.2mm m2")
@@
   (gr_rect (start 70.739 49.657) (end 84.709 63.627) (layer "Edge.Cuts") (width 0.1) (fill none))
   (gr_rect (start 94.615 106.807) (end 108.585 120.777) (layer "Edge.Cuts") (width 0.1) (fill none))
+  (gr_text "make sure m2 are where they need to be!" (at 113.665 131.953) (layer "F.Adhes")
+    (effects (font (size 1 1) (thickness 0.15)))
+  )
   (zone (net 0) (net_name "") (layers F&B.Cu) (hatch edge 0.508)
     (connect_pads (clearance 0.508))

Commit message: planning out m2 and relief cuts
Parts:
- moved REF** 1.63 mm to (46.5, 141.2)
Changed lines of the file:
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@@
   (net 0 "")
   (footprint "MountingHole:MountingHole_2.2mm_M2_Pad" (layer "F.Cu")
-    (at 47.752 140.208)
+    (at 46.482 141.224)
     (descr "Mounting Hole 2.2mm, M2")
     (tags "mounting hole 2.2mm m2")

Commit message: deleted unnecessary files
Parts:
- removed REF** (x4): MountingHole_2.2mm_M2_Pad, MountingHole:MountingHole_2.2mm_M2_Pad
- added H1: MountingHole, MountingHole:MountingHole_2.2mm_M2, F.Cu at (68.3, 49.8)
- added H2: MountingHole, MountingHole:MountingHole_2.2mm_M2, F.Cu at (220.7, 49.8)
- added H3: MountingHole, MountingHole:MountingHole_2.2mm_M2, F.Cu at (46.0, 141.2)
- added H4: MountingHole, MountingHole:MountingHole_2.2mm_M2, F.Cu at (244.5, 141.2)
- added H5: MountingHole, MountingHole:MountingHole_2.2mm_M2, F.Cu at (96.8, 147.6)
- added H6: MountingHole, MountingHole:MountingHole_2.2mm_M2, F.Cu at (192.1, 147.6)
- added MX52: MX-NoLED, MX_Only:MXOnly-2.75U-Hotswap, F.Cu at (118.3, 161.3)
- added MX53: MX-NoLED, MX_Only:MXOnly-6U-Centered-Hotswap, F.Cu at (149.2, 160.3)
- added MX54: MX-NoLED, MX_Only:MXOnly-2.25U-Hotswap, F.Cu at (165.9, 160.3)
- added MX55: MX-NoLED, MX_Only:MXOnly-1U-Hotswap, F.Cu at (196.8, 160.3)
- moved G*** 13.0 mm to (147.6, 79.4)
Other:
- outline, holes or cut-outs redrawn
- board text added: "add standoffs for stability?"
- board text added: "add the pcb cut outs for bottom mounting"
- board text removed: "make sure m2 are where they need to be!"

Commit message: pcb, plate cleaned
stabs reversed
Parts:
- MX52: footprint MX_Only:MXOnly-2.75U-Hotswap -> MX_Only:MXOnly-2.75U-Hotswap-ReversedStabilizers
- MX53: footprint MX_Only:MXOnly-6U-Centered-Hotswap -> MX_Only:MXOnly-6U-Centered-Hotswap-ReversedStabilizers
- MX54: footprint MX_Only:MXOnly-2.25U-Hotswap -> MX_Only:MXOnly-2.25U-Hotswap-ReversedStabilizers
- moved H3 2.63 mm to (43.8, 139.8)
- moved H4 1.52 mm to (244.5, 139.7)
- moved MX52 1.24 mm to (117.5, 160.3)
- moved MX53 1.14 mm to (148.3, 159.7)
- moved MX54 0.76 mm to (165.1, 160.3)
Other:
- board size 241.6 x 96.9 mm -> 241.6 x 95.4 mm

Commit message: edgecut pcb updated, switchplate updated
Parts:
- removed MX52: MX-NoLED, MX_Only:MXOnly-2.75U-Hotswap-ReversedStabilizers
- removed MX53: MX-NoLED, MX_Only:MXOnly-6U-Centered-Hotswap-ReversedStabilizers
- removed MX54: MX-NoLED, MX_Only:MXOnly-2.25U-Hotswap-ReversedStabilizers
- removed MX55: MX-NoLED, MX_Only:MXOnly-1U-Hotswap
- moved H4 19.1 mm to (263.5, 139.8)
- moved H3 18.5 mm to (25.3, 139.7)
- moved G*** 3.55 mm to (146.1, 76.2)
- moved H5 1.59 mm to (96.8, 146.1)
- moved H6 1.59 mm to (192.1, 146.1)
Other:
- board size 241.6 x 95.4 mm -> 243.4 x 95.4 mm
- board text added: "the PETER"
