File: the PETER switchplate.kicad_pcb (KiCad board)
At the start: 2 copper layers, 243.4 x 95.4 mm, 7 parts

Commit message: changing silkscreen to fit edge cuts
for production files
Parts:
- removed H5, H6: MountingHole, MountingHole:MountingHole_2.2mm_M2
- moved G*** 19.1 mm to (144.5, 95.2)
