File: Project/the PETER keyboard STM.kicad_pcb (KiCad board)
At the start: 2 copper layers, 238.2 x 95.4 mm, 142 parts, among them J3 USB_C_Receptacle_USB2.0, SW1 RotaryEncoder_Switch, SW12 RotaryEncoder_Switch, SW3 SKQGABE010, U2 STM32F072C8Tx, U3 XC6206PxxxMR-Regulator_Linear, U4 USBLC6-2SC6

Commit message: stm revision
Parts:
- moved C9 19.9 mm to (154.0, 58.7), turned to -90 degrees
- moved U3 17.9 mm to (151.6, 58.7), turned to 180 degrees
- moved C8 16.4 mm to (149.2, 58.7), turned to -90 degrees
- moved G*** 13.0 mm to (80.2, 87.2)
- moved G*** 7.09 mm to (146.8, 87.2)
- moved C3 1.88 mm to (146.6, 102.1)
- moved C7 1.88 mm to (147.6, 102.1)
- moved SW3 1.10 mm to (161.9, 93.7)
- moved C2 0.80 mm to (141.3, 94.5)
- moved R1 0.71 mm to (157.9, 93.7)
- moved C1 0.31 mm to (145.0, 87.9)
Connections:
- D37 pad 1:  ROW3 -> ROW3
- D38 pad 1:  ROW3 -> ROW3
- D39 pad 1:  ROW3 -> ROW3
- D40 pad 1:  ROW3 -> ROW3
- D41 pad 1:  ROW3 -> ROW3
- D42 pad 1:  ROW3 -> ROW3
- D43 pad 1:  ROW3 -> ROW3
- D44 pad 1:  ROW3 -> ROW3
- D45 pad 1:  ROW3 -> ROW3
- D46 pad 1:  ROW3 -> ROW3
- D47 pad 1:  ROW3 -> ROW3
- D48 pad 1:  ROW3 -> ROW3
- U2 pad 10: unconnected-(U2-PA0-Pad10) -> COL8
- U2 pad 11: ROW0 -> COL7
- U2 pad 12: rG -> COL6
- U2 pad 13: rH -> unconnected-(U2-PA3-Pad13)
- U2 pad 14: ROW4 -> unconnected-(U2-PA4-Pad14)
- U2 pad 15: COL1 -> unconnected-(U2-PA5-Pad15)
- U2 pad 16: COL0 -> unconnected-(U2-PA6-Pad16)
- U2 pad 17: rE -> COL5
- U2 pad 18: rF -> COL4
- U2 pad 19: rA -> COL3
- U2 pad 2: ROW1 -> ROTARY_D
- U2 pad 20: rB -> COL2
- U2 pad 21: ROW3 -> COL1
- U2 pad 22: unconnected-(U2-PB11-Pad22) -> COL0
- U2 pad 25: unconnected-(U2-PB12-Pad25) -> ROW3
- U2 pad 26: unconnected-(U2-PB13-Pad26) -> ROW4
- U2 pad 27: unconnected-(U2-PB14-Pad27) -> ROW0
- U2 pad 28: unconnected-(U2-PB15-Pad28) -> ROW1
- U2 pad 29: unconnected-(U2-PA8-Pad29) -> ROW2
- U2 pad 3: COL11 -> ROTARY_C
- U2 pad 30: unconnected-(U2-PA9-Pad30) -> ROTARY_A
- U2 pad 31: unconnected-(U2-PA10-Pad31) -> ROTARY_B
- U2 pad 37: COL10 -> unconnected-(U2-PA14-Pad37)
- U2 pad 38: COL9 -> unconnected-(U2-PA15-Pad38)
- U2 pad 39: COL8 -> unconnected-(U2-PB3-Pad39)
- U2 pad 4: ROW2 -> COL11
- U2 pad 40: COL7 -> unconnected-(U2-PB4-Pad40)
- U2 pad 41: COL6 -> unconnected-(U2-PB5-Pad41)
- U2 pad 42: COL5 -> unconnected-(U2-PB6-Pad42)
- U2 pad 43: COL4 -> unconnected-(U2-PB7-Pad43)
- U2 pad 45: COL3 -> unconnected-(U2-PB8-Pad45)
- U2 pad 46: COL2 -> unconnected-(U2-PB9-Pad46)
- U2 pad 5: rC -> COL10
- U2 pad 6: rD -> COL9
Routing:
- net ROW1: track 7.32 -> 378.6 mm, vias 0 -> 4
- net ROW3: track 0.00 -> 370.7 mm
- net ROW0: track 48.7 -> 392.6 mm
- net GND: track 36.0 -> 375.6 mm, vias 15 -> 17
- net  ROW3: track 303.1 -> 0.00 mm
- net ROW2: track 414.5 -> 216.6 mm, vias 0 -> 4
- net ROW4: track 206.0 -> 391.1 mm
- net COL0: track 80.0 -> 200.3 mm
- net Net-(D58-A): track 125.3 -> 7.71 mm
- net COL1: track 86.4 -> 175.3 mm
- net COL2: track 85.1 -> 156.5 mm
- net COL9: track 83.7 -> 145.7 mm
- net (no net): track 56.9 -> 0.00 mm
- net COL3: track 64.7 -> 117.9 mm
- net COL7: track 155.6 -> 119.9 mm
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Other:
- board size 238.2 x 95.4 mm -> 243.3 x 95.4 mm
- board text added: "MX1"
- board text added: "the PETER v2.0 by Calvin#0563"
- board text removed: "MOVE CUT OUT ON EDGES FOR FULL CASE COMPATIBILITZ (HEAT INSERT)"
- board text removed: "the PETER v1.0 by Calvin#0563"
